File: mainboard/main.sch (KiCad schematic (older format))
At the start: 55 parts, among them J1 USB_OTG, J2 HIB, J3 JTAG Port, J4 C Port, J5 A Port, J6 E Port, J7 D Port, J8 B Port, J9 F Port, SW1 SW_Push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

Commit message: Updated
Parts:
- C10: footprint tm4c:CP_Elec_4x5.4 -> Capacitor_Tantalum_SMD:CP_EIA-6032-20_AVX-F_Pad2.25x2.35mm_HandSolder
- C12: footprint tm4c:CP_Elec_4x5.4 -> Capacitor_Tantalum_SMD:CP_EIA-7343-30_AVX-N_Pad2.25x2.55mm_HandSolder
- Y1: footprint Crystal:Crystal_SMD_EuroQuartz_MT-4Pin_3.2x2.5mm_HandSoldering -> Crystal:Crystal_SMD_EuroQuartz_MJ-4Pin_5.0x3.2mm
Other:
- note added: "Read carefully PCB design for tiva series before layout"
- note added: "Use Tantalum to optimize the layout\n(C10;C12)"
Changed lines of the file:
@@
 PE3
-Wire Notes Line
-	11200 550  11200 4850
 Wire Notes Line
 	9100 550  9100 4850
@@
 F 0 "C10" H 3800 1350 50  0000 L CNN
 F 1 "10uF" H 3750 1200 50  0000 L CNN
-F 2 "tm4c:CP_Elec_4x5.4" H 4038 1150 50  0001 C CNN
+F 2 "Capacitor_Tantalum_SMD:CP_EIA-6032-20_AVX-F_Pad2.25x2.35mm_HandSolder" H 4038 1150 50  0001 C CNN
 F 3 "~" H 4000 1300 50  0001 C CNN
 	1    4000 1300
@@
 F 0 "C12" H 4650 1350 50  0000 L CNN
 F 1 "22uF" H 4600 1200 50  0000 L CNN
-F 2 "tm4c:CP_Elec_4x5.4" H 4888 1150 50  0001 C CNN
+F 2 "Capacitor_Tantalum_SMD:CP_EIA-7343-30_AVX-N_Pad2.25x2.55mm_HandSolder" H 4888 1150 50  0001 C CNN
 F 3 "~" H 4850 1300 50  0001 C CNN
 	1    4850 1300
@@
 $EndComp
 $Comp
-L power:+3.3V #PWR?
-U 1 1 5EFC274D
-P 11000 1175
-AR Path="/5DC79FAF/5EFC274D" Ref="#PWR?"  Part="1"
-AR Path="/5EFC274D" Ref="#PWR051"  Part="1"
-F 0 "#PWR051" H 11000 1025 50  0001 C CNN
-F 1 "+3.3V" H 11100 1325 50  0000 C CNN
-F 2 "" H 11000 1175 50  0001 C CNN
-F 3 "" H 11000 1175 50  0001 C CNN
-	1    11000 1175
-	1    0    0    -1
-$EndComp
-$Comp
 L power:+5V #PWR?
 U 1 1 5EFC2A69
@@
 Wire Wire Line
 	2010 4900 3050 4900
-Entry Wire Line
-	4560 2200 4660 2300
 Wire Wire Line
 	3750 2000 3750 1950
@@
 F 0 "Y1" H 2354 5446 50  0000 L CNN
 F 1 "Crystal_GND24_Small" H 2354 5355 50  0000 L CNN
-F 2 "Crystal:Crystal_SMD_EuroQuartz_MT-4Pin_3.2x2.5mm_HandSoldering" H 2210 5400 50  0001 C CNN
+F 2 "Crystal:Crystal_SMD_EuroQuartz_MJ-4Pin_5.0x3.2mm" H 2210 5400 50  0001 C CNN
 F 3 "~" H 2210 5400 50  0001 C CNN
 	1    2210 5400
@@
 Wire Wire Line
 	2210 5230 2540 5230
+Text Notes 4040 740  0    50   ~ 0
+Use Tantalum to optimize the layout\n(C10;C12)
+Wire Notes Line
+	11200 550  11200 4850
+Text Notes 6970 6430 0    50   ~ 0
+Read carefully PCB design for tiva series before layout
 $EndSCHEMATC

Commit message: Updated v1.3
Parts:
- C10: footprint Capacitor_Tantalum_SMD:CP_EIA-6032-20_AVX-F_Pad2.25x2.35mm_HandSolder -> tm4c:tantalum6032
- C12: footprint Capacitor_Tantalum_SMD:CP_EIA-7343-30_AVX-N_Pad2.25x2.55mm_HandSolder -> tm4c:tantalum7343
- Y1: footprint Crystal:Crystal_SMD_EuroQuartz_MJ-4Pin_5.0x3.2mm -> tm4c:Crystal_SMD_5032-4Pin_5.0x3.2mm
- Y2: footprint Crystal:Crystal_SMD_MicroCrystal_CC7V-T1A-2Pin_3.2x1.5mm_HandSoldering -> tm4c:Crystal_SMD_MicroCrystal_CC7V-T1A-2Pin_3.2x1.5mm_HandSoldering
Other:
- note removed: "Read carefully PCB design for tiva series before layout"
- moved on the sheet: C1, C11, C14, C15, C16, C17, C18, C2, C3, C4, C5, C6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

Commit message: Updated
Parts:
- removed J4: C Port, tm4c:PinHeader_1x10_P2.54mm_Vertical, symbol Connector:Conn_01x10_Male
- removed J5: A Port, tm4c:PinHeader_1x10_P2.54mm_Vertical, symbol Connector:Conn_01x10_Male
- removed J6: E Port, tm4c:PinHeader_1x10_P2.54mm_Vertical, symbol Connector:Conn_01x10_Male
- removed J7: D Port, tm4c:PinHeader_1x10_P2.54mm_Vertical, symbol Connector:Conn_01x10_Male
- removed J8: B Port, tm4c:PinHeader_1x10_P2.54mm_Vertical, symbol Connector:Conn_01x10_Male
- removed J9: F Port, tm4c:PinHeader_1x10_P2.54mm_Vertical, symbol Connector:Conn_01x10_Male
- added J1, J2: 2x10 male, Connector_PinHeader_2.54mm:PinHeader_2x10_P2.54mm_Vertical_SMD, symbol Connector_Generic:Conn_02x10_Counter_Clockwise
Connections:
- net D+: no longer J1.3 (D+)
- net D-: no longer J1.2 (D-)
- net PA0: now also J1.1 (Pin_1)
- net PA1: now also J1.2 (Pin_2)
- net PA2: now also J1.3 (Pin_3)
- net PA3: now also J1.4 (Pin_4)
- net PA4: now also J1.5 (Pin_5)
- net PA5: now also J1.6 (Pin_6)
- net PA6: now also J1.7 (Pin_7)
- net PA7: now also J1.8 (Pin_8)
- net PB0: now also J1.20 (Pin_20)
- net PB1: now also J1.19 (Pin_19)
- net PB2: now also J1.18 (Pin_18)
- net PB3: now also J1.17 (Pin_17)
- net PB4: now also J1.16 (Pin_16)
- net PB5: now also J1.15 (Pin_15)
- net PB6: now also J1.14 (Pin_14)
- net PB7: now also J1.13 (Pin_13)
- net PC4: now also J1.9 (Pin_9)
- net PC5: now also J1.10 (Pin_10)
- net PC6: now also J1.12 (Pin_12)
- net PC7: now also J1.11 (Pin_11)
- net PD0: now also J2.1 (Pin_1)
- net PD1: now also J2.2 (Pin_2)
- net PD2: now also J2.3 (Pin_3)
- net PD3: now also J2.4 (Pin_4)
- net PD6: now also J2.7 (Pin_7)
- net PD7: now also J2.8 (Pin_8)
- net PE0: now also J2.20 (Pin_20)
- net PE1: now also J2.19 (Pin_19)
- net PE2: now also J2.18 (Pin_18)
- net PE3: now also J2.17 (Pin_17)
- net PE4: now also J2.16 (Pin_16)
- net PE5: now also J2.15 (Pin_15)
- net PF0: now also J2.9 (Pin_9)
- net PF1: now also J2.10 (Pin_10)
- net PF2: now also J2.14 (Pin_14)
- net PF3: now also J2.13 (Pin_13)
- net PF4: now also J2.12 (Pin_12)
- new net PD4-: J1.2 (D-), J2.5 (Pin_5)
- new net PD5+: J1.3 (D+), J2.6 (Pin_6)
